File: pcb/mx/plate/plate.kicad_sch (KiCad schematic)
At the start: 66 parts, among them SW1 SW_PUSH, SW10 SW_PUSH, SW11 SW_PUSH, SW12 SW_PUSH, SW13 SW_PUSH, SW14 SW_PUSH, SW15 SW_PUSH, SW16 SW_PUSH, SW17 SW_PUSH, SW18 SW_PUSH, SW19 SW_PUSH, SW2 SW_PUSH, SW20 SW_PUSH, SW21 SW_PUSH, SW22 SW_PUSH, SW23 SW_PUSH, SW24 SW_PUSH, SW25 SW_PUSH, SW26 SW_PUSH, SW27 SW_PUSH, SW28 SW_PUSH, SW29 SW_PUSH, SW3 SW_PUSH, SW30 SW_PUSH, SW31 SW_PUSH, SW4 SW_PUSH, SW5 SW_PUSH, SW6 SW_PUSH, SW7 SW_PUSH, SW8 SW_PUSH, SW9 SW_PUSH

Commit message: Fix 微調整
Parts:
- added H5, H6, H7, H8: MountingHole, 0_kbd:M2_HOLE_v3, symbol Mechanical:MountingHole
Changed lines of the file:
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@@
+    )
+  )
+  (symbol (lib_id "Mechanical:MountingHole") (at 205.74 153.67 0) (unit 1)
+    (in_bom yes) (on_board yes) (dnp no) (fields_autoplaced)
+    (property "Reference" "H8" (at 208.28 152.4579 0)
+      (effects (font (size 1.27 1.27)) (justify left))
+    )
+    (property "Value" "MountingHole" (at 208.28 154.8821 0)
+      (effects (font (size 1.27 1.27)) (justify left))
+    )
+    (property "Footprint" "0_kbd:M2_HOLE_v3" (at 205.74 153.67 0)
+      (effects (font (size 1.27 1.27)) hide)
+    )
+    (property "Datasheet" "~" (at 205.74 153.67 0)
+      (effects (font (size 1.27 1.27)) hide)
+    )
+    (instances
+      (project "plate"
+        (path "/6e471c34-fb9c-4836-aac9-8239f9e8a673"
+          (reference "H8") (unit 1)
+        )
+      )
     )
   )
@@
         (path "/6e471c34-fb9c-4836-aac9-8239f9e8a673"
           (reference "H1") (unit 1)
+        )
+      )
+    )
+  )
+  (symbol (lib_id "Mechanical:MountingHole") (at 205.74 148.59 0) (unit 1)
+    (in_bom yes) (on_board yes) (dnp no) (fields_autoplaced)
+    (property "Reference" "H7" (at 208.28 147.3779 0)
+      (effects (font (size 1.27 1.27)) (justify left))
+    )
+    (property "Value" "MountingHole" (at 208.28 149.8021 0)
+      (effects (font (size 1.27 1.27)) (justify left))
+    )
+    (property "Footprint" "0_kbd:M2_HOLE_v3" (at 205.74 148.59 0)
+      (effects (font (size 1.27 1.27)) hide)
+    )
+    (property "Datasheet" "~" (at 205.74 148.59 0)
+      (effects (font (size 1.27 1.27)) hide)
+    )
+    (instances
+      (project "plate"
+        (path "/6e471c34-fb9c-4836-aac9-8239f9e8a673"
+          (reference "H7") (unit 1)
         )
       )
@@
     )
   )
+  (symbol (lib_id "Mechanical:MountingHole") (at 205.74 138.43 0) (unit 1)
+    (in_bom yes) (on_board yes) (dnp no) (fields_autoplaced)
+    (property "Reference" "H5" (at 208.28 137.2179 0)
+      (effects (font (size 1.27 1.27)) (justify left))
+    )
+    (property "Value" "MountingHole" (at 208.28 139.6421 0)
+      (effects (font (size 1.27 1.27)) (justify left))
+    )
+    (property "Footprint" "0_kbd:M2_HOLE_v3" (at 205.74 138.43 0)
+      (effects (font (size 1.27 1.27)) hide)
+    )
+    (property "Datasheet" "~" (at 205.74 138.43 0)
+      (effects (font (size 1.27 1.27)) hide)
+    )
+    (instances
+      (project "plate"
+        (path "/6e471c34-fb9c-4836-aac9-8239f9e8a673"
+          (reference "H5") (unit 1)
+        )
+      )
+    )
+  )
   (symbol (lib_id "Device:D") (at 148.59 135.89 90) (unit 1)
     (in_bom yes) (on_board yes) (dnp no) (fields_autoplaced)
@@
         )
       )
+    )
+  )
+  (symbol (lib_id "Mechanical:MountingHole") (at 205.74 143.51 0) (unit 1)
+    (in_bom yes) (on_board yes) (dnp no) (fields_autoplaced)
+    (property "Reference" "H6" (at 208.28 142.2979 0)
+      (effects (font (size 1.27 1.27)) (justify left))
+    )
+    (property "Value" "MountingHole" (at 208.28 144.7221 0)
+      (effects (font (size 1.27 1.27)) (justify left))
+    )
+    (property "Footprint" "0_kbd:M2_HOLE_v3" (at 205.74 143.51 0)
+      (effects (font (size 1.27 1.27)) hide)
+    )
+    (property "Datasheet" "~" (at 205.74 143.51 0)
+      (effects (font (size 1.27 1.27)) hide)
+    )
+    (instances
+      (project "plate"
+        (path "/6e471c34-fb9c-4836-aac9-8239f9e8a673"
+          (reference "H6") (unit 1)
+        )
+      )
