File: pcb/mx/plate/plate.kicad_pcb (KiCad board)
At the start: 2 copper layers, 133.3 x 113.3 mm, 36 parts, among them SW1 SW_PUSH, SW10 SW_PUSH, SW11 SW_PUSH, SW12 SW_PUSH, SW13 SW_PUSH, SW14 SW_PUSH, SW15 SW_PUSH, SW16 SW_PUSH, SW17 SW_PUSH, SW18 SW_PUSH, SW19 SW_PUSH, SW2 SW_PUSH, SW20 SW_PUSH, SW21 SW_PUSH, SW22 SW_PUSH, SW23 SW_PUSH, SW24 SW_PUSH, SW25 SW_PUSH, SW26 SW_PUSH, SW27 SW_PUSH, SW28 SW_PUSH, SW29 SW_PUSH, SW3 SW_PUSH, SW30 SW_PUSH, SW31 SW_PUSH, SW4 SW_PUSH, SW5 SW_PUSH, SW6 SW_PUSH, SW7 SW_PUSH, SW8 SW_PUSH, SW9 SW_PUSH

Commit message: Fix 微調整
Parts:
- added H3: MountingHole, 0_kbd:M2_HOLE_v3, F.Cu at (180.1, 98.7)
- added H3: MountingHole, 0_kbd:M2_HOLE_v3, F.Cu at (84.8, 24.8)
- added H3: MountingHole, 0_kbd:M2_HOLE_v3, F.Cu at (84.8, 108.6)
- added H3: MountingHole, 0_kbd:M2_HOLE_v3, F.Cu at (180.1, 32.0)
- moved H1 14.2 mm to (166.7, 103.8)
- moved REF** 9.53 mm to (65.8, 104.8)
Other:
- outline, holes or cut-outs redrawn

Commit message: release: sage60 v0.0.1
Other:
- outline, holes or cut-outs redrawn
Changed lines of the file:
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@@
     )
     (pad_to_mask_clearance 0)
-    (grid_origin 180.07 98.687573)
+    (grid_origin 180.07 83.447573)
     (pcbplotparams
       (layerselection 0x0001000_7ffffffe)
@@
       (drillshape 0)
       (scaleselection 1)
-      (outputdirectory "/Users/daiki/Projects/sage60/pcb/mx/plate/")
+      (outputdirectory "../../../../../Users/Daiki Iwamoto/Downloads/")
     )
   )
@@
     )
   )
+  (gr_line (start 189.54624 106.403993) (end 172.40124 98.783993)
+    (stroke (width 0.15) (type default)) (layer "Dwgs.User"))
   (gr_circle (center 180.07 98.687573) (end 181.07 98.687573)
     (stroke (width 0.1) (type default)) (fill none) (layer "Edge.Cuts"))
@@
   (gr_circle (center 84.82 24.765) (end 85.82 24.765)
     (stroke (width 0.1) (type default)) (fill none) (layer "Edge.Cuts"))
-  (gr_line (start 189.54624 106.403993) (end 189.595 35.822573)
+  (gr_line (start 189.54624 92.972573) (end 189.595 35.822573)
     (stroke (width 0.1) (type default)) (layer "Edge.Cuts"))
   (gr_line (start 177.07 35.822573) (end 170.545 35.822573)
@@
   (gr_circle (center 151.495 44.7675) (end 152.495 44.7675)
     (stroke (width 0.1) (type default)) (fill none) (layer "Edge.Cuts"))
+  (gr_line (start 189.54624 102.403993) (end 189.54624 106.403993)
+    (stroke (width 0.1) (type default)) (layer "Edge.Cuts"))
   (gr_line (start 189.595 35.822573) (end 183.07 35.822573)
     (stroke (width 0.1) (type default)) (layer "Edge.Cuts"))
@@
     (stroke (width 0.1) (type default)) (layer "Edge.Cuts"))
   (gr_line (start 94.345 116.205) (end 118.1575 116.205)
+    (stroke (width 0.1) (type default)) (layer "Edge.Cuts"))
+  (gr_line (start 182.9275 92.972573) (end 182.9275 102.403993)
     (stroke (width 0.1) (type default)) (layer "Edge.Cuts"))
   (gr_circle (center 96.25 97.155) (end 97.25 97.155)
@@
   (gr_line (start 81.82 108.585) (end 81.82 104.775)
     (stroke (width 0.1) (type default)) (layer "Edge.Cuts"))
+  (gr_line (start 182.9275 102.403993) (end 189.54624 102.403993)
+    (stroke (width 0.1) (type default)) (layer "Edge.Cuts"))
   (gr_line (start 94.345 104.775) (end 94.345 116.205)
     (stroke (width 0.1) (type default)) (layer "Edge.Cuts"))
@@
   (gr_circle (center 166.735 103.8225) (end 167.735 103.8225)
     (stroke (width 0.1) (type default)) (fill none) (layer "Edge.Cuts"))
+  (gr_line (start 182.9275 92.972573) (end 189.54624 92.972573)
+    (stroke (width 0.1) (type default)) (layer "Edge.Cuts"))
   (gr_line (start 67.675 108.585) (end 75.295 108.585)
     (stroke (width 0.1) (type default)) (layer "Edge.Cuts"))
