File: pcb/mx/daughter/daughter.kicad_pcb (KiCad board)
At the start: 2 copper layers, 71.4 x 46.4 mm, 7 parts, among them J1 MJ-4PP-9, J2 Conn_01x06_Socket, J3 Conn_01x06_Socket

Commit message: release: sage60 v0.0.1
Parts:
- added BAT+: Conn_01x01_Pin, kbd:1pin_conn, F.Cu at (137.0, -22.6)
- added BAT-: Conn_01x01_Pin, kbd:1pin_conn, F.Cu at (141.0, -22.6)
- added REF**: Breakaway_Tabs, kbd:Breakaway_Tabs, F.Cu at (138.7, -9.26)
- added SW32: SW_SPDT, Connector_PinHeader_2.54mm:PinHeader_1x03_P2.54mm_Vertical, F.Cu at (124.5, -27.6)
- moved J1 19.1 mm to (161.0, -29.3)
- moved H6 18.1 mm to (151.2, -26.4)
- moved RESET1 2.25 mm to (108.0, -27.7)
Routing:
- net RAW: track 19.6 -> 52.2 mm
- net +3.3V: track 70.1 -> 89.1 mm
- net Net-(J6-Pin_1): track 0.00 -> 14.6 mm
- net GND: track 0.00 -> 5.95 mm
- net RESET: track 25.9 -> 28.1 mm
Other:
- board size 71.4 x 46.4 mm -> 90.5 x 46.4 mm
- board text added: "JLCJLCJLCJLC"
