File: pcb/mx/daughter/daughter.kicad_sch (KiCad schematic)
At the start: 75 parts, among them J1 MJ-4PP-9, J2 Conn_01x06_Socket, J3 Conn_01x06_Socket, J4 Conn_01x06_Pin, J5 Conn_01x06_Pin, SW1 SW_PUSH, SW10 SW_PUSH, SW11 SW_PUSH, SW12 SW_PUSH, SW13 SW_PUSH, SW14 SW_PUSH, SW15 SW_PUSH, SW16 SW_PUSH, SW17 SW_PUSH, SW18 SW_PUSH, SW19 SW_PUSH, SW2 SW_PUSH, SW20 SW_PUSH, SW21 SW_PUSH, SW22 SW_PUSH, SW23 SW_PUSH, SW24 SW_PUSH, SW25 SW_PUSH, SW26 SW_PUSH, SW27 SW_PUSH, SW28 SW_PUSH, SW29 SW_PUSH, SW3 SW_PUSH, SW30 SW_PUSH, SW31 SW_PUSH, SW4 SW_PUSH, SW5 SW_PUSH, SW6 SW_PUSH, SW7 SW_PUSH, SW8 SW_PUSH, SW9 SW_PUSH

Commit message: release: sage60 v0.0.1
Parts:
- added J6: Conn_01x01_Pin, kbd:1pin_conn, symbol Connector:Conn_01x01_Pin
- added SW32: SW_SPDT, Connector_PinHeader_2.54mm:PinHeader_1x03_P2.54mm_Vertical, symbol Switch:SW_SPDT
Connections:
- net RAW: now also SW32.2 (B)
- new net: J6.1 (Pin_1), SW32.1 (A)
- no-connect marks 6 -> 7
