File: pcb/poc/poc.kicad_pcb (KiCad board)
At the start: 2 copper layers, 81 x 83 mm, 19 parts, among them J1 MJ-4PP-9, SW00 EC_SW, SW01 EC_SW, SW10 EC_SW, SW11 EC_SW, U2 OPA350, U3 74HC4051

Commit message: release: sage60 v0.0.1
Parts:
- U2: value OPA350 -> TLV9061IDBVR; footprint Package_SO:SOIC-8_3.9x4.9mm_P1.27mm -> Package_TO_SOT_SMD:SOT-23-5
- moved U2 1.31 mm to (111.6, 73.6)
Connections:
- U2 pad 1: (no net) -> Net-(JP1-B)
- U2 pad 2: Net-(JP1-B) -> GND
- U2 pad 4: GND -> ADC
- U2 pad 5: (no net) -> POWER
Routing:
- net GND: vias 8 -> 18
