File: pcb/mx_right_tb/mx_right_tb.kicad_pcb (KiCad board)
At the start: 2 copper layers, 134.9 x 111.5 mm, 60 parts, among them SW1 SW_PUSH, SW10 SW_PUSH, SW11 SW_PUSH, SW12 SW_PUSH, SW13 SW_PUSH, SW14 SW_PUSH, SW15 SW_PUSH, SW16 SW_PUSH, SW17 SW_PUSH, SW18 SW_PUSH, SW19 SW_PUSH, SW2 SW_PUSH, SW20 SW_PUSH, SW21 SW_PUSH, SW22 SW_PUSH, SW23 SW_PUSH, SW24 SW_PUSH, SW27 SW_PUSH, SW28 SW_PUSH, SW29 SW_PUSH, SW3 SW_PUSH, SW30 SW_PUSH, SW32 SW_SPDT, SW4 SW_PUSH, SW5 SW_PUSH, SW6 SW_PUSH, SW7 SW_PUSH, SW8 SW_PUSH, SW9 SW_PUSH

Commit message: modify
Parts:
- moved J1 5.54 mm to (161.0, 122.4)
Routing:
- net SDIO: track 158.9 -> 164.4 mm
- net SCLK: track 158.4 -> 164.0 mm
- net MOTION: track 157.1 -> 162.7 mm
- net 3.3V: track 188.2 -> 193.7 mm
- net CS: track 169.0 -> 174.5 mm
- net COL3: track 233.0 -> 232.1 mm
Other:
- board size 134.9 x 111.5 mm -> 134.9 x 113.3 mm
