File: pcb/mx_right_tb/mx_right_tb.kicad_pcb (KiCad board)
At the start: 2 copper layers, 134.9 x 113.3 mm, 60 parts, among them SW1 SW_PUSH, SW10 SW_PUSH, SW11 SW_PUSH, SW12 SW_PUSH, SW13 SW_PUSH, SW14 SW_PUSH, SW15 SW_PUSH, SW16 SW_PUSH, SW17 SW_PUSH, SW18 SW_PUSH, SW19 SW_PUSH, SW2 SW_PUSH, SW20 SW_PUSH, SW21 SW_PUSH, SW22 SW_PUSH, SW23 SW_PUSH, SW24 SW_PUSH, SW27 SW_PUSH, SW28 SW_PUSH, SW29 SW_PUSH, SW3 SW_PUSH, SW30 SW_PUSH, SW32 SW_SPDT, SW4 SW_PUSH, SW5 SW_PUSH, SW6 SW_PUSH, SW7 SW_PUSH, SW8 SW_PUSH, SW9 SW_PUSH

Commit message: feat: order-ready MX boards (phi 5 centre holes), separate left / right plates, case updates
- PCBs: switch centre holes phi 4.1 -> 5 for Kailh Choc v2 (centre_hole.py); the tracks that fell
  inside the new hole clearance are rerouted by centre_reroute.py (grid A*, vias where one layer is
  full). DRC errors unchanged, 0 unconnected, schematic parity as before.
- SW32 stays a 3-pin THT footprint (2.54 mm); the case's knob opening follows its middle pin
  (SW_Y -54.86) and the finger scoop sits 1 mm toward +y to avoid a thin wall at the MCU block.
- Plates: one per side (pcb/mx_left_plate, pcb/mx_right_tb_plate) instead of the shared
  breakaway plate; 1.2 mm 3MFs for test prints.
- Top case: chamfer on the top outer edge (top_chamfer); machinability probe fix.
- Regenerated specs, 3MFs and MCU cover DXFs; all four documents pass check.py,
  check_parts.py and machinability.py.

Co-Authored-By: Claude Opus 5.5 <noreply@anthropic.com>
Routing:
- net SCLK: track 164.0 -> 182.3 mm, vias 1 -> 7
- net SDIO: track 169.1 -> 178.4 mm, vias 2 -> 4
- net MOTION: track 166.5 -> 175.3 mm
- net CS: track 174.5 -> 178.0 mm, vias 1 -> 3

Commit message: feat(case): magnets hold the trackball case; MCU cover magnet; J1 pin socket
- trackball case: the two M1.7 screw bosses grow to r3.75 and take a
  phi6x3 magnet from below (tb_socket_cut.py); the bottom case gets
  facing phi6.1x3.1 holes in the seat (TB_MAGS / TB_MAG_CUT) instead of
  the through holes and desk-side counterbores
- MCU cover held by one magnet in a top case boss + steel disc
- J1: round-pin socket + cut-down L header (tongue_socket.py, stage6
  J1_REF), trackball case hood cut for it; LP J1_RELIEF
- re-exported right 3MFs and MCU cover DXFs

Co-Authored-By: Claude Opus 5.5 <noreply@anthropic.com>
Parts:
- moved J1 5.64 mm to (166.6, 122.4)
Routing:
- net 3.3V: track 193.7 -> 197.2 mm
- net MOTION: track 175.3 -> 177.9 mm
- net SCLK: track 182.3 -> 184.6 mm
- net CS: track 178.0 -> 180.2 mm, vias 3 -> 4
- net SDIO: track 178.4 -> 180.4 mm
Other:
- outline, holes or cut-outs redrawn
Changed lines of the file:
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@@
 	(footprint "0_sora:pmw3610_connector"
 		(layer "F.Cu")
-		(at 160.995 122.395)
+		(at 166.64 122.395)
 		(property "Reference" "J1"
 			(at 0 -0.5 0)
@@
 	(gr_line
 		(start 159.9 105.775)
-		(end 159.9 131.315)
+		(end 159.9 111.8)
 		(stroke
 			(width 0.1)
@@
 	)
 	(gr_arc
-		(start 160.9 132.315)
-		(mid 160.192893 132.022107)
-		(end 159.9 131.315)
+		(start 160.9 112.8)
+		(mid 160.192893 112.507107)
+		(end 159.9 111.8)
 		(stroke
 			(width 0.1)
@@
 	)
 	(gr_line
-		(start 165.931632 132.315)
-		(end 160.9 132.315)
+		(start 160.9 112.8)
+		(end 162.4 112.8)
+		(stroke
+			(width 0.1)
+			(type default)
+		)
+		(layer "Edge.Cuts")
+	)
+	(gr_arc
+		(start 162.4 112.8)
+		(mid 163.107107 113.092893)
+		(end 163.4 113.8)
+		(stroke
+			(width 0.1)
+			(type default)
+		)
+		(layer "Edge.Cuts")
+	)
+	(gr_line
+		(start 163.4 113.8)
+		(end 163.4 131.315)
+		(stroke
+			(width 0.1)
+			(type default)
+		)
+		(layer "Edge.Cuts")
+	)
+	(gr_arc
+		(start 164.4 132.315)
+		(mid 163.692893 132.022107)
+		(end 163.4 131.315)
+		(stroke
+			(width 0.1)
+			(type default)
+		)
+		(layer "Edge.Cuts")
+	)
+	(gr_line
+		(start 173 132.315)
+		(end 164.4 132.315)
+		(stroke
+			(width 0.1)
+			(type default)
+		)
+		(layer "Edge.Cuts")
+	)
+	(gr_arc
+		(start 174 116.839204)
+		(mid 174.027984 116.60429)
+		(end 174.110369 116.382524)
+		(stroke
+			(width 0.1)
+			(type default)
+		)
+		(layer "Edge.Cuts")
+	)
+	(gr_arc
+		(start 174 131.315)
+		(mid 173.707107 132.022107)
+		(end 173 132.315)
+		(stroke
+			(width 0.1)
+			(type default)
+		)
+		(layer "Edge.Cuts")
+	)
+	(gr_line
+		(start 174 131.315)
+		(end 174 116.839204)
 		(stroke
 			(width 0.1)
@@
 	(gr_line
 		(start 180.06647 104.779824)
-		(end 165.931632 132.315)
+		(end 174.110369 116.382524)
 		(stroke
 			(width 0.1)
@@
 	)
 	(segment
+		(start 166.64 113.945)
+		(end 166.64 114.775)
+		(width 0.25)
+		(layer "B.Cu")
+		(net "SCLK")
+	)
+	(segment
 		(start 156.745 77.875)
 		(end 158.595 79.725)
@@
 	)
 	(segment
+		(start 160.995 108.3)
+		(end 166.64 113.945)
+		(width 0.25)
+		(layer "B.Cu")
+		(net "SCLK")
+	)
+	(segment
 		(start 160.995 105.775)
 		(end 157.995 102.775)
@@
 	)
 	(segment
+		(start 160.995 105.775)
+		(end 160.995 108.3)
+		(width 0.25)
+		(layer "B.Cu")
+		(net "SCLK")
+	)
+	(segment
 		(start 158.995 49.775)
 		(end 159.495 50.275)
@@
 	)
 	(segment
-		(start 160.995 114.775)
-		(end 160.995 105.775)
-		(width 0.25)
-		(layer "B.Cu")
-		(net "SCLK")
-	)
-	(segment
 		(start 157.995 94.5767)
 		(end 157.995 95.4416)
@@
 	)
 	(segment
+		(start 164.71835 107.5)
+		(end 164.71835 117.315)
+		(width 0.25)
+		(layer "F.Cu")
+		(net "CS")
+	)
+	(segment
+		(start 164.71835 117.315)
+		(end 166.64 117.315)
+		(width 0.25)
+		(layer "F.Cu")
+		(net "CS")
+	)
+	(segment
 		(start 111.995 44.775)
 		(end 113.995 44.775)
@@
 		(net "CS")
 	)
-	(segment
-		(start 162.495 105.27665)
-		(end 162.495 115.815)
-		(width 0.25)
-		(layer "B.Cu")
+	(via
+		(at 164.71835 107.5)
+		(size 0.8)
+		(drill 0.4)
+		(layers "F.Cu" "B.Cu")
 		(net "CS")
 	)
@@
 	)
 	(segment
-		(start 162.495 115.815)
-		(end 160.995 117.315)
+		(start 163.945 77.4566)
+		(end 163.945 74.1566)
 		(width 0.25)
 		(layer "B.Cu")
@@
 	)
 	(segment
-		(start 163.945 77.4566)
-		(end 163.945 74.1566)
+		(start 160.245 80.1066)
+		(end 161.295 80.1066)
 		(width 0.25)
 		(layer "B.Cu")
@@
 	)
 	(segment
-		(start 160.245 80.1066)
-		(end 161.295 80.1066)
+		(start 162.495 105.27665)
+		(end 164.71835 107.5)
 		(width 0.25)
 		(layer "B.Cu")
@@
 	)
 	(segment
-		(start 170.495 112.895)
-		(end 170.495 101.775)
+		(start 173 122.395)
+		(end 166.64 122.395)
+		(width 0.5)
+		(layer "B.Cu")
+		(net "3.3V")
+	)
+	(segment
+		(start 170.495 105.3)
+		(end 173 107.805)
+		(width 0.5)
+		(layer "B.Cu")
+		(net "3.3V")
+	)
+	(segment
+		(start 173 107.805)
+		(end 173 122.395)
 		(width 0.5)
 		(layer "B.Cu")
@@
 	)
 	(segment
+		(start 170.495 101.775)
+		(end 170.495 105.3)
+		(width 0.5)
+		(layer "B.Cu")
+		(net "3.3V")
+	)
+	(segment
 		(start 72.520004 80.275)
 		(end 75.795 83.549996)
@@
 	)
 	(segment
-		(start 160.995 122.395)
-		(end 170.495 112.895)
-		(width 0.5)
-		(layer "B.Cu")
-		(net "3.3V")
+		(start 163.95 127.475)
+		(end 166.64 127.475)
+		(width 0.25)
+		(layer "F.Cu")
+		(net "SDIO")
 	)
 	(segment
@@
 	)
 	(segment
-		(start 163.3 104.791493)
-		(end 163.3 125.17)
-		(width 0.25)
-		(layer "F.Cu")
-		(net "SDIO")
-	)
-	(segment
 		(start 100.2467 52.9075)
 		(end 101.7967 52.9075)
@@
 	)
 	(segment
+		(start 163.95 112.15)
+		(end 163.95 127.475)
+		(width 0.25)
+		(layer "F.Cu")
+		(net "SDIO")
+	)
+	(segment
+		(start 163.3 104.791493)
+		(end 163.3 111.5)
+		(width 0.25)
+		(layer "F.Cu")
+		(net "SDIO")
+	)
+	(segment
 		(start 97.821167 51.8075)
 		(end 99.14665 51.8075)
@@
 	)
 	(segment
-		(start 163.3 125.17)
-		(end 160.995 127.475)
-		(width 0.25)
-		(layer "F.Cu")
-		(net "SDIO")
-	)
-	(segment
 		(start 158.795 103.791493)
 		(end 162.3 103.791493)
@@
 		(net "SDIO")
 	)
+	(segment
+		(start 163.3 111.5)
+		(end 163.95 112.15)
+		(width 0.25)
+		(layer "F.Cu")
+		(net "SDIO")
+	)
 	(via
 		(at 139.495 97.779993)
@@
 	)
 	(segment
+		(start 162.45 104.841493)
+		(end 162.45 111.3)
+		(width 0.25)
+		(layer "F.Cu")
+		(net "MOTION")
+	)
+	(segment
 		(start 120.495 96.275)
 		(end 122.624993 98.404993)
@@
 		(net "MOTION")
 	)
-	(segment
-		(start 162.45 104.841493)
-		(end 162.45 124)
-		(width 0.25)
-		(layer "F.Cu")
-		(net "MOTION")
-	)
 	(via
-		(at 120.495 96.275)
+		(at 162.45 111.3)
 		(size 0.8)
 		(drill 0.4)
@@
 	)
 	(via
-		(at 162.45 124)
+		(at 120.495 96.275)
 		(size 0.8)
 		(drill 0.4)
@@
 	)
 	(segment
+		(start 164.2 113.05)
+		(end 164.2 130.015)
+		(width 0.25)
+		(layer "B.Cu")
+		(net "MOTION")
+	)
+	(segment
 		(start 124.195 88.649)
 		(end 125.845 86.999)
@@
 	)
 	(segment
-		(start 162.45 128.56)
-		(end 160.995 130.015)
+		(start 164.2 130.015)
+		(end 166.64 130.015)
 		(width 0.25)
 		(layer "B.Cu")
@@
 	)
 	(segment
-		(start 162.45 124)
-		(end 162.45 128.56)
+		(start 125.845 67.949)
+		(end 125.845 64.748999)
 		(width 0.25)
 		(layer "B.Cu")
@@
 	)
 	(segment
-		(start 125.845 67.949)
-		(end 125.845 64.748999)
+		(start 162.45 111.3)
+		(end 164.2 113.05)
 		(width 0.25)
 		(layer "B.Cu")
