File: pcb/mx_main/mx.kicad_pcb (KiCad board)
At the start: 2 copper layers, 134.9 x 111.5 mm, 63 parts, among them SW1 SW_PUSH, SW10 SW_PUSH, SW11 SW_PUSH, SW12 SW_PUSH, SW13 SW_PUSH, SW14 SW_PUSH, SW15 SW_PUSH, SW16 SW_PUSH, SW17 SW_PUSH, SW18 SW_PUSH, SW19 SW_PUSH, SW2 SW_PUSH, SW20 SW_PUSH, SW21 SW_PUSH, SW22 SW_PUSH, SW23 SW_PUSH, SW24 SW_PUSH, SW25 SW_PUSH, SW26 SW_PUSH, SW27 SW_PUSH, SW28 SW_PUSH, SW29 SW_PUSH, SW3 SW_PUSH, SW30 SW_PUSH, SW32 SW_SPDT, SW4 SW_PUSH, SW5 SW_PUSH, SW6 SW_PUSH, SW7 SW_PUSH, SW8 SW_PUSH, SW9 SW_PUSH

Commit message: feat: sage60 case generator, phi6 magnets and shared plate
- mechanical/case: scripts that build the split case (MX and low-profile) in Fusion from KiCad
  (outline, gasket shelf, USB-C, slide switch, MCU cover, trackball), with interference checks and
  PCB/switch/keycap reference models for renders
- top case: case A (skirt down to the desk); guards over the gaps between the main block, the thumb
  cluster and the right column; the bare PCB around the trackball is covered too
- magnets: Daiso phi6x3, 4 per side
- left PCB: reroute ROW4 near SW28 and add a semicircular edge notch for a magnet post
- plate: one plate for both halves; the right half snips off the trackball part (slots + bridges)
  and the front gasket tab (mouse bites) and is used flipped

Co-Authored-By: Claude Opus 5.5 <noreply@anthropic.com>
Routing:
- net ROW4: track 137.1 -> 141.4 mm, vias 4 -> 5
Other:
- outline, holes or cut-outs redrawn
Changed lines of the file:
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@@
 	(gr_line
 		(start 177.021746 129.927534)
+		(end 185.545349 109.428059)
+		(stroke
+			(width 0.1)
+			(type default)
+		)
+		(layer "Edge.Cuts")
+	)
+	(gr_arc
+		(start 185.545349 109.428059)
+		(mid 183.414595 104.264254)
+		(end 188.5784 102.133499)
+		(stroke
+			(width 0.1)
+			(type default)
+		)
+		(layer "Edge.Cuts")
+	)
+	(gr_line
+		(start 188.5784 102.133499)
 		(end 191.077007 96.124288)
 		(stroke
@@
 	)
 	(segment
+		(start 176.05 104)
+		(end 176.05 112.014)
+		(width 0.25)
+		(layer "F.Cu")
+		(net "ROW4")
+	)
+	(segment
 		(start 176.0505 112.013993)
 		(end 177.765 112.013993)
@@
 		(net "ROW4")
 	)
-	(segment
-		(start 189.604 73.91625)
-		(end 188.071 75.44925)
-		(width 0.25)
-		(layer "B.Cu")
+	(via
+		(at 176.05 104)
+		(size 0.8)
+		(drill 0.4)
+		(layers "F.Cu" "B.Cu")
 		(net "ROW4")
 	)
 	(segment
-		(start 187.977497 101.801497)
-		(end 177.765 112.013993)
+		(start 189.604 73.91625)
+		(end 188.071 75.44925)
 		(width 0.25)
 		(layer "B.Cu")
@@
 	)
 	(segment
+		(start 178.521 104)
+		(end 176.05 104)
+		(width 0.25)
+		(layer "B.Cu")
+		(net "ROW4")
+	)
+	(segment
 		(start 188.74824 93.77325)
 		(end 188.02224 94.49925)
@@
 	)
 	(segment
-		(start 188.02224 94.49925)
-		(end 188.02224 101.756754)
+		(start 188.022 94.4993)
+		(end 178.521 104)
 		(width 0.25)
 		(layer "B.Cu")
@@
 	)
 	(segment
-		(start 188.02224 101.756754)
-		(end 187.977497 101.801497)
+		(start 177.765 112.013993)
+		(end 179.345 110.495)
 		(width 0.25)
 		(layer "B.Cu")
@@
 		(width 0.25)
 		(layer "B.Cu")
-		(net "ROW4")
-	)
-	(segment
-		(start 188.02224 101.756753)
-		(end 187.977497 101.801497)
-		(width 0.25)
-		(layer "B.Cu")
